Commit message: working plugin

File: extended_robot_hw_tests/test/urdf/extended_simple_transmission_loader.urdf (robot description, URDF)
Before this commit: robot robot, 0 links, 0 joints
Links:
- added link link_1
- added link link_2
Joints:
- added joint extended_joint: type floating, parent link_1, child link_2
